File: Nyan Mouse/HW/Board/fpga_not_sane.sch (KiCad schematic (older format))
At the start: 0 parts

Commit message: Added all FPGA parts and updated excel sheet of pinout.
Parts:
- added IC? (x9): ep4ce15e22c8n, symbol ep4ce15e22c8n
Connections:
- new net +1.2V: IC?.102 (VCCINT), IC?.116 (VCCINT), IC?.124 (VCCINT), IC?.138 (VCCINT), IC?.29 (VCCINT), IC?.34 (VCCINT), IC?.38 (VCCINT), IC?.45 (VCCINT), IC?.5 (VCCINT), IC?.70 (VCCINT), IC?.78 (VCCINT), IC?.84 (VCCINT)
- new net +2.5V: IC?.107 (VCCA2), IC?.3 (VCCA3), IC?.35 (VCCA1), IC?.75 (VCCA4)
- new net +3.3VD: IC?.117 (VCCIO7), IC?.122 (VCCIO7), IC?.130 (VCCIO8), IC?.139 (VCCIO8), IC?.17 (VCCIO1), IC?.26 (VCCIO2), IC?.40 (VCCIO3), IC?.47 (VCCIO3), IC?.56 (VCCIO4), IC?.62 (VCCIO4), IC?.81 (VCCIO5), IC?.93 (VCCIO6)
- new net AGND: IC?.108 (GNDA2), IC?.2 (GNDA3), IC?.36 (GNDA1), IC?.74 (GNDA4)
- new net DGND: IC?.118 (GND), IC?.123 (GND), IC?.131 (GND), IC?.140 (GND), IC?.19 (GND), IC?.22 (GND), IC?.27 (GND), IC?.4 (GND), IC?.41 (GND), IC?.48 (GND), IC?.57 (GND), IC?.63 (GND), IC?.79 (GND), IC?.82 (GND), IC?.95 (GND)
- new net VDD: IC?.1 (VCCD_PLL3), IC?.109 (VCCD_PLL2), IC?.37 (VCCD_PLL1), IC?.73 (VCCD_PLL4)
