File: Nyan Mouse/HW/Board/fpga_not_sane.sch (KiCad schematic (older format))
At the start: 9 parts

Commit message: Schematic things have been updated
Parts:
- removed IC? (x4): ep4ce15e22c8n, symbol ep4ce15e22c8n
- added C? (x11): 0.1uF, symbol Csmall
- added C? (x8): 1uF, symbol Csmall
- added C? (x5): 10uF, symbol Csmall
- added C? (x3): 100uF, symbol CP1
- added L?: 10nH, symbol INDUCTOR_SMALL
Connections:
- net +1.2V: now also C?.1, C?.1, C?.1, C?.1, C?.1, C?.1, C?.1, C?.1, C?.1, C?.1, C?.1, C?.1, C?.1
- net +2.5V: now also C?.1, C?.1, C?.1, L?.2
- net +3.3VD: now also C?.1, C?.1, C?.1, C?.1, C?.1, C?.1, C?.1
- net AGND: now also C?.2, C?.2, C?.2, C?.2
- net DGND: now also C?.2, C?.2, C?.2, C?.2, C?.2, C?.2, C?.2, C?.2, C?.2, C?.2, C?.2, C?.2, C?.2, C?.2, C?.2, C?.2, C?.2, C?.2, C?.2, C?.2, C?.2, C?.2, C?.2
- net VDD: now also C?.1, C?.1, C?.1, C?.1, L?.1
Other:
- note added: "place all of these capacitors near the fpga"
