File: Nyan Mouse/HW/Board/fpga/fpga_bank_5_6.sch (KiCad schematic (older format))
At the start: 0 parts

Commit message: Added ESD prevention documentation.
Added ByteBlaster documentation.

Modified FPGA banks.
Parts:
- added IC? (x2): ep4ce15e22c8n, symbol ep4ce15e22c8n
Changed lines of the file:
@@
 LIBS:contrib
 LIBS:valves
+LIBS:ip4221cz6-s
+LIBS:3v3custom
+LIBS:adc128s052
+LIBS:altera_ep4ce15e22c
+LIBS:drv8837
+LIBS:JST-XH-BattBalance
+LIBS:lp3987
+LIBS:mic94345-4ycs
+LIBS:s25fl064p
+LIBS:SparkFun
+LIBS:stm32f103rx
+LIBS:tps6205x
 LIBS:Nyan Mouse Daughter-cache
 EELAYER 24 0
 EELAYER END
-$Descr A4 11693 8268
+$Descr USLetter 11000 8500
 encoding utf-8
-Sheet 1 4
+Sheet 4 5
 Title ""
 Date ""
@@
 Comment4 ""
 $EndDescr
+$Comp
+L ep4ce15e22c8n IC?
+U 6 1 535B103B
+P 3350 4050
+F 0 "IC?" H 3350 4100 60  0000 C CNN
+F 1 "ep4ce15e22c8n" H 3350 4000 60  0000 C CNN
+F 2 "" H 3350 4050 60  0000 C CNN
+F 3 "" H 3350 4050 60  0000 C CNN
+	6    3350 4050
+	1    0    0    -1
+$EndComp
+$Comp
+L ep4ce15e22c8n IC?
+U 7 1 535B104F
+P 7600 4100
+F 0 "IC?" H 7600 4150 60  0000 C CNN
+F 1 "ep4ce15e22c8n" H 7600 4050 60  0000 C CNN
+F 2 "" H 7600 4100 60  0000 C CNN
+F 3 "" H 7600 4100 60  0000 C CNN
+	7    7600 4100
+	1    0    0    -1
+$EndComp
 $EndSCHEMATC
