File: Nyan Mouse/HW/Board/fpga/fpga_bank_7_8.sch (KiCad schematic (older format))
At the start: 0 parts

Commit message: Added ESD prevention documentation.
Added ByteBlaster documentation.

Modified FPGA banks.
Parts:
- added IC? (x2): ep4ce15e22c8n, symbol ep4ce15e22c8n
Changed lines of the file:
@@
 LIBS:contrib
 LIBS:valves
+LIBS:ip4221cz6-s
+LIBS:3v3custom
+LIBS:adc128s052
+LIBS:altera_ep4ce15e22c
+LIBS:drv8837
+LIBS:JST-XH-BattBalance
+LIBS:lp3987
+LIBS:mic94345-4ycs
+LIBS:s25fl064p
+LIBS:SparkFun
+LIBS:stm32f103rx
+LIBS:tps6205x
 LIBS:Nyan Mouse Daughter-cache
 EELAYER 24 0
 EELAYER END
-$Descr A4 11693 8268
+$Descr USLetter 11000 8500
 encoding utf-8
-Sheet 1 1
+Sheet 5 5
 Title ""
 Date ""
@@
 Comment4 ""
 $EndDescr
+$Comp
+L ep4ce15e22c8n IC?
+U 8 1 535B106D
+P 3400 4150
+F 0 "IC?" H 3400 4200 60  0000 C CNN
+F 1 "ep4ce15e22c8n" H 3400 4100 60  0000 C CNN
+F 2 "" H 3400 4150 60  0000 C CNN
+F 3 "" H 3400 4150 60  0000 C CNN
+	8    3400 4150
+	1    0    0    -1
+$EndComp
+$Comp
+L ep4ce15e22c8n IC?
+U 9 1 535B1081
+P 7700 4200
+F 0 "IC?" H 7700 4250 60  0000 C CNN
+F 1 "ep4ce15e22c8n" H 7700 4150 60  0000 C CNN
+F 2 "" H 7700 4200 60  0000 C CNN
+F 3 "" H 7700 4200 60  0000 C CNN
+	9    7700 4200
+	1    0    0    -1
+$EndComp
 $EndSCHEMATC
