File: Nyan Mouse/HW/Board/fpga/Nyan Mouse Daughter.sch (KiCad schematic (older format))
At the start: 45 parts

Commit message: Updated schematics
Parts:
- C? (x4): value 0.1uF -> 0.01uF
- C? (x4): value 10nF -> 0.1uF
- C? (x7): value Csmall -> 10pF
Changed lines of the file:
@@
 P 3150 6550
 F 0 "C?" H 3175 6600 30  0000 L CNN
-F 1 "0.1uF" H 3175 6500 30  0000 L CNN
+F 1 "0.01uF" H 3175 6500 30  0000 L CNN
 F 2 "" H 3150 6550 60  0000 C CNN
 F 3 "" H 3150 6550 60  0000 C CNN
@@
 P 3350 6550
 F 0 "C?" H 3375 6600 30  0000 L CNN
-F 1 "0.1uF" H 3375 6500 30  0000 L CNN
+F 1 "0.01uF" H 3375 6500 30  0000 L CNN
 F 2 "" H 3350 6550 60  0000 C CNN
 F 3 "" H 3350 6550 60  0000 C CNN
@@
 P 3350 6900
 F 0 "C?" H 3375 6950 30  0000 L CNN
-F 1 "0.1uF" H 3375 6850 30  0000 L CNN
+F 1 "0.01uF" H 3375 6850 30  0000 L CNN
 F 2 "" H 3350 6900 60  0000 C CNN
 F 3 "" H 3350 6900 60  0000 C CNN
@@
 P 3150 6900
 F 0 "C?" H 3175 6950 30  0000 L CNN
-F 1 "0.1uF" H 3175 6850 30  0000 L CNN
+F 1 "0.01uF" H 3175 6850 30  0000 L CNN
 F 2 "" H 3150 6900 60  0000 C CNN
 F 3 "" H 3150 6900 60  0000 C CNN
@@
 P 7100 6400
 F 0 "C?" H 7100 6500 40  0000 L CNN
-F 1 "10nF" H 7106 6315 40  0000 L CNN
+F 1 "0.1uF" H 7106 6315 40  0000 L CNN
 F 2 "" H 7138 6250 30  0000 C CNN
 F 3 "" H 7100 6400 60  0000 C CNN
@@
 P 8700 6400
 F 0 "C?" H 8700 6500 40  0000 L CNN
-F 1 "10nF" H 8706 6315 40  0000 L CNN
+F 1 "0.1uF" H 8706 6315 40  0000 L CNN
 F 2 "" H 8738 6250 30  0000 C CNN
 F 3 "" H 8700 6400 60  0000 C CNN
@@
 P 10350 6300
 F 0 "C?" H 10350 6400 40  0000 L CNN
-F 1 "10nF" H 10356 6215 40  0000 L CNN
+F 1 "0.1uF" H 10356 6215 40  0000 L CNN
 F 2 "" H 10388 6150 30  0000 C CNN
 F 3 "" H 10350 6300 60  0000 C CNN
@@
 P 9050 6300
 F 0 "C?" H 9050 6400 40  0000 L CNN
-F 1 "10nF" H 9056 6215 40  0000 L CNN
+F 1 "0.1uF" H 9056 6215 40  0000 L CNN
 F 2 "" H 9088 6150 30  0000 C CNN
 F 3 "" H 9050 6300 60  0000 C CNN
@@
 P 4500 5200
 F 0 "C?" H 4525 5250 30  0000 L CNN
-F 1 "Csmall" H 4525 5150 30  0000 L CNN
+F 1 "10pF" H 4525 5150 30  0000 L CNN
 F 2 "" H 4500 5200 60  0000 C CNN
 F 3 "" H 4500 5200 60  0000 C CNN
@@
 P 4600 5400
 F 0 "C?" H 4625 5450 30  0000 L CNN
-F 1 "Csmall" H 4625 5350 30  0000 L CNN
+F 1 "10pF" H 4625 5350 30  0000 L CNN
 F 2 "" H 4600 5400 60  0000 C CNN
 F 3 "" H 4600 5400 60  0000 C CNN
@@
 P 4700 5200
 F 0 "C?" H 4725 5250 30  0000 L CNN
-F 1 "Csmall" H 4725 5150 30  0000 L CNN
+F 1 "10pF" H 4725 5150 30  0000 L CNN
 F 2 "" H 4700 5200 60  0000 C CNN
 F 3 "" H 4700 5200 60  0000 C CNN
@@
 P 4800 5400
 F 0 "C?" H 4825 5450 30  0000 L CNN
-F 1 "Csmall" H 4825 5350 30  0000 L CNN
+F 1 "10pF" H 4825 5350 30  0000 L CNN
 F 2 "" H 4800 5400 60  0000 C CNN
 F 3 "" H 4800 5400 60  0000 C CNN
@@
 P 4900 5200
 F 0 "C?" H 4925 5250 30  0000 L CNN
-F 1 "Csmall" H 4925 5150 30  0000 L CNN
+F 1 "10pF" H 4925 5150 30  0000 L CNN
 F 2 "" H 4900 5200 60  0000 C CNN
 F 3 "" H 4900 5200 60  0000 C CNN
@@
 P 5000 5400
 F 0 "C?" H 5025 5450 30  0000 L CNN
-F 1 "Csmall" H 5025 5350 30  0000 L CNN
+F 1 "10pF" H 5025 5350 30  0000 L CNN
 F 2 "" H 5000 5400 60  0000 C CNN
 F 3 "" H 5000 5400 60  0000 C CNN
@@
 P 5100 5200
 F 0 "C?" H 5125 5250 30  0000 L CNN
-F 1 "Csmall" H 5125 5150 30  0000 L CNN
+F 1 "10pF" H 5125 5150 30  0000 L CNN
 F 2 "" H 5100 5200 60  0000 C CNN
 F 3 "" H 5100 5200 60  0000 C CNN
